File: PCB/Untitled.kicad_sch (KiCad schematic)
At the start: 5 parts, among them J1 DEBUG, J2 USB_C_Receptacle_PowerOnly_6P, U1 74HC4051, U2 74HC4051

Commit message: something works
Parts:
- removed J1: DEBUG, symbol Connector_Generic_MountingPin:Conn_01x03_MountingPin
- removed J2: USB_C_Receptacle_PowerOnly_6P, symbol Connector:USB_C_Receptacle_PowerOnly_6P
- removed U1: 74HC4051, symbol 74xx:74HC4051
- added J1: LCD, symbol Connector_Generic_MountingPin:Conn_01x04_MountingPin
- added J2: BELL, symbol Connector_Generic_MountingPin:Conn_01x02_MountingPin
Connections:
- net at U2.10 (S1): now also A1.27 (GPIO21)
- net at U2.11 (S0): now also A1.29 (GPIO22)
- net +3V3: now reaches U2.16 (VCC)
- net +3V3: now also A1.36 (3V3)
- net at U2.3 (A): now also A1.31 (GPIO26_ADC0)
- net GND: now reaches U2.6 (~{E})
- net GND: now also A1.13 (GND), A1.18 (GND), A1.23 (GND), A1.28 (GND), A1.3 (GND), A1.38 (GND), A1.8 (GND), U2.7 (VEE), U2.8 (GND), J1.1 (Pin_1), J2.2 (Pin_2)
- net at U2.9 (S2): now also A1.26 (GPIO20)
- net at A1.16 (GPIO12): now also J1.3 (Pin_3)
- net at A1.17 (GPIO13): now also J1.4 (Pin_4)
- net at A1.2 (GPIO1): now also J2.1 (Pin_1)
- net +5V: now reaches A1.40 (VBUS)
- net +5V: now also J1.2 (Pin_2)
Other:
- moved on the sheet: U2

Commit message: pcb
Parts:
- removed J1: LCD, symbol Connector_Generic_MountingPin:Conn_01x04_MountingPin
- removed J2: BELL, symbol Connector_Generic_MountingPin:Conn_01x02_MountingPin
- added J1: LCD, Connector_PinHeader_2.54mm:PinHeader_1x04_P2.54mm_Vertical, symbol Connector:Conn_01x04_Pin
- added J2: HORN, Connector_PinHeader_2.54mm:PinHeader_1x02_P2.54mm_Vertical, symbol Connector:Conn_01x02_Pin
- added J3: BELL, Connector_PinHeader_2.54mm:PinHeader_1x02_P2.54mm_Vertical, symbol Connector:Conn_01x02_Pin
- U2: footprint (none) -> Package_DIP:DIP-16_W7.62mm
Connections:
- net +5V: now also J1.3 (Pin_3)
- net GND: now also A1.33 (AGND), J1.4 (Pin_4), J2.1 (Pin_1), J3.1 (Pin_1)
- net at A1.2 (GPIO1): now also J2.2 (Pin_2)
- net at A1.16 (GPIO12): now also J1.2 (Pin_2)
- net at A1.17 (GPIO13): now also J1.1 (Pin_1)
- net at A1.4 (GPIO2): now also J3.2 (Pin_2)
